File: Hardware/Schematic_openbook v62.brd (EAGLE design)
At the start: 170.2 x 111.2 mm, 103 parts, among them IC1 BD5229G-TR, IC4 XC6220A331MR-G, J1 FH34SRJ-24S-0.5SH_99_, J2 SAMACSYS_PARTS_USB4110-GF-A, J3 QWIIC_RIGHT_ANGLE, J4 112A-TAAR-R03_ATTEND, Q1 20V/4.2A/52mΩ/1.4W, Q2 20V/4.2A/52mΩ/1.4W, Q3 SI1308EDL-T1-GE3, U1 W25Q512JVEIQ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

Commit message: Fixed (Review #1)
Parts:
- CHG_LED, SJ1: value (none) -> NA
- moved C10_SUPERCAP 23.6 mm to (94.8, 60.9), turned to 180 degrees
- moved C8 14.9 mm to (94.3, 65.3), turned to 0 degrees
- moved D1 1.44 mm to (155.0, 52.0), turned to 0 degrees
Connections:
- net DN: now also D1.4; no longer D1.1
- net DP: now also D1.6; no longer D1.3
- net GND: now also D1.2; no longer D1.5
- net USB_D+: now also D1.1; no longer D1.4
- net USB_D-: now also D1.3; no longer D1.6
- net VBUS: now also D1.5; no longer D1.2
Routing:
- net VRTC: track 25.3 -> 31.1 mm
- net USB_D-: track 137.7 -> 139.1 mm
- net USB_D+: track 134.8 -> 136.1 mm
- net DP: track 12.2 -> 11.0 mm
- net DN: track 12.9 -> 11.9 mm
