File: Hardware/Schematic_openbook_v58.sch (EAGLE design)
At the start: 103 parts, among them IC1 BD5229G-TR, IC4 XC6220A331MR-G, J1 FH34SRJ-24S-0.5SH_99_, J2 SAMACSYS_PARTS_USB4110-GF-A, J3 QWIIC_RIGHT_ANGLE, J4 112A-TAAR-R03_ATTEND, Q1 20V/4.2A/52mΩ/1.4W, Q2 20V/4.2A/52mΩ/1.4W, Q3 SI1308EDL-T1-GE3, U1 W25Q512JVEIQ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

Commit message: Fixed (Review #1)
Parts:
- CHG_LED, SJ1: value (none) -> NA
Connections:
- net DN: now also D1.I/O2_2; no longer D1.I/O1_1
- net DP: now also D1.I/O1_2; no longer D1.I/O2_1
- net GND: now also D1.GND; no longer D1.VBUS
- net USB_D+: now also D1.I/O1_1; no longer D1.I/O2_2
- net USB_D-: now also D1.I/O2_1; no longer D1.I/O1_2
- net VBUS: now also D1.VBUS; no longer D1.GND
Other:
- moved on the sheet: D1
